File: kicad6_files/gba_flex_ds_lite/gba_flex_ds_lite.kicad_pcb (KiCad board)
At the start: 2 copper layers, 58 x 16.4 mm, 4 parts, among them J1 Conn_01x32, J2 Conn_01x32, U1 KDSO643, U2 KDSO643

Commit message: updated board and gerbers files to latest version
Routing:
- net Net-(J1-Pad32): track 12.0 -> 18.4 mm, vias 0 -> 1
- net Net-(J1-Pad31): track 12.0 -> 16.3 mm, vias 0 -> 1
Other:
- outline, holes or cut-outs redrawn
- board text added: "Facelesstech 2023 DS_Lite_GBA_Slot_Flex rev C"
- board text removed: "Facelesstech 2022 DS_Lite_GBA_Slot_Flex rev B"
